File: Hardware/JankPad/top_PCB_v2.brd (EAGLE design)
At the start: 126 x 67.5 mm, 7 parts, among them X1 FH12-40S-0.5SH

Commit message: more bugs
Parts:
- moved X1 1.61 mm to (65.0, 33.9), turned to 270 degrees
Routing:
- net N$31: track 192.6 -> 225.2 mm, vias 4 -> 8
- net N$2: track 92.0 -> 114.7 mm, vias 4 -> 6
- net N$12: track 35.7 -> 55.9 mm
- net N$10: track 31.3 -> 48.4 mm, vias 1 -> 2
- net N$11: track 34.2 -> 50.0 mm, vias 1 -> 2
- net N$1: track 40.9 -> 52.4 mm, vias 1 -> 2
- net N$8: track 91.5 -> 101.2 mm, vias 1 -> 2
- net N$27: track 70.7 -> 79.8 mm, vias 1 -> 2
- net N$26: track 59.0 -> 67.7 mm, vias 1 -> 2
- net N$25: track 55.7 -> 64.0 mm, vias 1 -> 2
- net N$24: track 53.4 -> 61.1 mm, vias 1 -> 2
- net N$22: track 46.2 -> 52.9 mm, vias 1 -> 2
- net N$21: track 67.3 -> 73.6 mm, vias 1 -> 2
- net N$18: track 55.4 -> 60.7 mm, vias 1 -> 2
- net N$17: track 52.4 -> 57.5 mm, vias 1 -> 2
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