File: Hardware/JankPad-StopGap/top_PCB_mini.sch (EAGLE design)
At the start: 7 parts

Commit message: Snapshot!!
Connections:
- removed net N$28: LAUNCHPAD.PB6, LEFTJOYSTICK.X
- removed net N$34: LAUNCHPAD.PB7, LEFTJOYSTICK.Y
- new net N$10: LAUNCHPAD.PB6
- new net N$11: LAUNCHPAD.PD2, LEFTJOYSTICK.X
- new net N$12: LAUNCHPAD.PD3, LEFTJOYSTICK.Y
Changed lines of the file:
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@@
-</segment>
-</net>
-<net name="N$28" class="0">
-<segment>
-<pinref part="LEFTJOYSTICK" gate="G$1" pin="X"/>
-<wire x1="-27.94" y1="5.08" x2="-40.64" y2="5.08" width="0.1524" layer="91"/>
-<pinref part="LAUNCHPAD" gate="G$1" pin="PB6"/>
-<wire x1="106.68" y1="7.62" x2="109.22" y2="7.62" width="0.1524" layer="91"/>
-<wire x1="109.22" y1="7.62" x2="109.22" y2="-53.34" width="0.1524" layer="91"/>
-<wire x1="109.22" y1="-53.34" x2="-40.64" y2="-53.34" width="0.1524" layer="91"/>
-<wire x1="-40.64" y1="-53.34" x2="-40.64" y2="5.08" width="0.1524" layer="91"/>
 </segment>
 </net>
@@
 <pinref part="LAUNCHPAD" gate="G$1" pin="PF4"/>
 <wire x1="127" y1="-17.78" x2="106.68" y2="-17.78" width="0.1524" layer="91"/>
-</segment>
-</net>
-<net name="N$34" class="0">
-<segment>
-<pinref part="LEFTJOYSTICK" gate="G$1" pin="Y"/>
-<wire x1="-15.24" y1="25.4" x2="0" y2="25.4" width="0.1524" layer="91"/>
-<wire x1="0" y1="25.4" x2="0" y2="-55.88" width="0.1524" layer="91"/>
-<wire x1="0" y1="-55.88" x2="119.38" y2="-55.88" width="0.1524" layer="91"/>
-<wire x1="119.38" y1="-55.88" x2="119.38" y2="17.78" width="0.1524" layer="91"/>
-<pinref part="LAUNCHPAD" gate="G$1" pin="PB7"/>
-<wire x1="119.38" y1="17.78" x2="106.68" y2="17.78" width="0.1524" layer="91"/>
 </segment>
 </net>
@@
 </segment>
 </net>
+<net name="N$10" class="0">
+<segment>
+<pinref part="LAUNCHPAD" gate="G$1" pin="PB6"/>
+<wire x1="106.68" y1="7.62" x2="109.22" y2="7.62" width="0.1524" layer="91"/>
+</segment>
+</net>
+<net name="N$11" class="0">
+<segment>
+<pinref part="LEFTJOYSTICK" gate="G$1" pin="X"/>
+<wire x1="-27.94" y1="5.08" x2="-43.18" y2="5.08" width="0.1524" layer="91"/>
+<wire x1="-43.18" y1="5.08" x2="-43.18" y2="-25.4" width="0.1524" layer="91"/>
+<wire x1="-43.18" y1="-25.4" x2="35.56" y2="-25.4" width="0.1524" layer="91"/>
+<wire x1="35.56" y1="-25.4" x2="35.56" y2="27.94" width="0.1524" layer="91"/>
+<pinref part="LAUNCHPAD" gate="G$1" pin="PD2"/>
+<wire x1="35.56" y1="27.94" x2="50.8" y2="27.94" width="0.1524" layer="91"/>
+</segment>
+</net>
+<net name="N$12" class="0">
+<segment>
+<pinref part="LAUNCHPAD" gate="G$1" pin="PD3"/>
+<wire x1="50.8" y1="17.78" x2="5.08" y2="17.78" width="0.1524" layer="91"/>
+<wire x1="5.08" y1="17.78" x2="5.08" y2="30.48" width="0.1524" layer="91"/>
+<pinref part="LEFTJOYSTICK" gate="G$1" pin="Y"/>
+<wire x1="5.08" y1="30.48" x2="-15.24" y2="30.48" width="0.1524" layer="91"/>
+<wire x1="-15.24" y1="30.48" x2="-15.24" y2="25.4" width="0.1524" layer="91"/>
+</segment>
+</net>
